Commit message: La costmap fonctionne les marker de mppi sont a régler prochainement

File: src/robot_description/urdf/robot.xacro (robot description, xacro)
@@ -125,7 +125,7 @@
     </link>
 <joint name="base_footprint_joint" type="fixed">
-<parent link="base_link"/>
-<child link="base_footprint"/>
-<origin xyz="0 0 0" rpy="0 0 0"/>
+<parent link="base_footprint"/>
+<child link="base_link"/>
+<origin xyz="0 0 0" rpy="0 0 1.5708"/>
 <axis xyz="0 0 1"/>
 </joint>

Commit message: MPPI commence a etre ok prochaine etape : corriger le urdf car peut etre inversion d'axe

File: src/robot_description/urdf/robot.xacro (robot description, xacro)
@@ -134,5 +134,5 @@
     <parent link="base_link"/>
     <child link="laser_frame"/>
-    <origin xyz="0 0 0.075" rpy="0 0 0"/>
+    <origin xyz="0 0 0.075" rpy="0 0 1.5708"/>
     <axis xyz="0 0 1"/>
 </joint>

Commit message: La nav confiture ptn de merde faut regler la précision et les vitesse

File: src/robot_description/urdf/robot.xacro (robot description, xacro)
@@ -7,6 +7,6 @@
   <inertial>
     <origin xyz="-0.00014980415129537406 0.0003023390699038116 0.0332081283017649" rpy="0 0 0"/>
-    <mass value="6.063579487839896"/>
-    <inertia ixx="0.0277" iyy="0.022027" izz="0.038299" ixy="-0.0" iyz="0.000161" ixz="-1e-06"/>
+    <mass value="0.063579487839896"/>
+    <inertia ixx="0.000277" iyy="0.00022027" izz="0.00038299" ixy="-0.0" iyz="0.000161" ixz="-1e-06"/>
   </inertial>
   <visual>
@@ -27,5 +27,5 @@
   <inertial>
     <origin xyz="-0.0010380506382758475 -1.1679208535467223e-05 -2.1888176668372061e-07" rpy="0 0 0"/>
-    <mass value="0.6461883281506762"/>
+    <mass value="0.06461883281506762"/>
     <inertia ixx="0.000287" iyy="0.00019" izz="0.00019" ixy="0.0" iyz="-0.0" ixz="0.0"/>
   </inertial>
@@ -47,5 +47,5 @@
   <inertial>
     <origin xyz="-0.0010380506382763194 -1.1679208533246777e-05 -2.188817664235121e-07" rpy="0 0 0"/>
-    <mass value="0.6461883281506762"/>
+    <mass value="0.06461883281506762"/>
     <inertia ixx="0.000287" iyy="0.00019" izz="0.00019" ixy="0.0" iyz="0.0" ixz="0.0"/>
   </inertial>
@@ -67,5 +67,5 @@
   <inertial>
     <origin xyz="0.001038572809780841 1.1096913653231566e-05 -2.1888178453749463e-07" rpy="0 0 0"/>
-    <mass value="0.646188328150675"/>
+    <mass value="0.0646188328150675"/>
     <inertia ixx="0.000287" iyy="0.00019" izz="0.00019" ixy="0.0" iyz="0.0" ixz="0.0"/>
   </inertial>
@@ -87,5 +87,5 @@
   <inertial>
     <origin xyz="0.0010385728097805635 1.1096913650872342e-05 -2.188817843883084e-07" rpy="0 0 0"/>
-    <mass value="0.6461883281506752"/>
+    <mass value="0.06461883281506752"/>
     <inertia ixx="0.000287" iyy="0.00019" izz="0.00019" ixy="0.0" iyz="0.0" ixz="0.0"/>
   </inertial>
